File: USB-C-HYBRID/K02-USB-C-HYBRID.kicad_pcb (KiCad board)
At the start: 2 copper layers, 109.4 x 86.9 mm, 28 parts, among them SW1 SW_Push, SW10 SW_Push, SW11 SW_Push, SW12 SW_Push, SW13 SW_Push, SW14 SW_Push, SW15 SW_Push, SW16 SW_Push, SW17 SW_Push, SW2 SW_Push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

Commit message: almost there
Routing:
- net Switch2: track 94.9 -> 97.4 mm
- net Switch12: track 82.6 -> 84.4 mm
- net raw: track 55.6 -> 56.6 mm
- net BT+_r: track 58.8 -> 59.8 mm
- net Switch6: track 126.7 -> 127.6 mm
- net Switch3: track 73.0 -> 73.6 mm
- net Switch7: track 84.4 -> 85.0 mm
